Commit message: switch gripper

File: ur_robot_server/urdf/Robotiq85/urRobotiq85_macro.xacro (robot description, xacro)
@@ -59,6 +59,18 @@
       safety_k_position="${safety_k_position}"
     />
-    <xacro:include filename="$(find ur_robot_server)/urdf/Robotiq85/couplerRobotiq.xacro"/>
-    <xacro:robotiq_coupler_macro />
+    <!--
+      Import the xacro macro for the REAL robotiq gripper (augmented with Gazebo
+      specific elements in the respective repo).
+    -->
+    <xacro:include filename="$(find robotiq_2f_85_gripper_visualization)/urdf/robotiq_arg2f_85_model_macro.xacro"/>
+    <!-- Instantiate model for the gripper-->
+    <!-- robotiq 2f 85 gripper -->
+    <xacro:robotiq_arg2f_85 prefix=""/>
+    <!-- attaches the gripper to the ur end effector -->
+    <joint name="gripper_ur5_joint" type="fixed">
+        <parent link="tool0"/>
+        <child link="robotiq_arg2f_base_link"/>
+        <origin xyz="0 0 0.01" rpy="0 0 0"/>
+    </joint>
     <!-- Configure self collision properties per link -->
     <gazebo reference="${prefix}shoulder_link">

Commit message: accepts 85 or 140 grippers

File: ur_robot_server/urdf/Robotiq85/urRobotiq85_macro.xacro (robot description, xacro)
@@ -38,5 +38,6 @@
    visual_parameters_file
    transmission_hw_interface:=hardware_interface/EffortJointInterface
-   safety_limits:=false safety_pos_margin:=0.15 safety_k_position:=20"
+   safety_limits:=false safety_pos_margin:=0.15 safety_k_position:=20
+   gripper_model"
   >
     <!--
@@ -62,15 +63,45 @@
       Import the xacro macro for the REAL robotiq gripper (augmented with Gazebo
       specific elements in the respective repo).
+      Picks between the 85 and 140 models
     -->
-    <xacro:include filename="$(find robotiq_2f_85_gripper_visualization)/urdf/robotiq_arg2f_85_model_macro.xacro"/>
-    <!-- Instantiate model for the gripper-->
-    <!-- robotiq 2f 85 gripper -->
-    <xacro:robotiq_arg2f_85 prefix=""/>
-    <!-- attaches the gripper to the ur end effector -->
+    <!-- If model 85-->
+    <xacro:if value="${gripper_model == 85}">
+      <xacro:include filename="$(find robotiq_2f_85_gripper_visualization)/urdf/robotiq_arg2f_85_model_macro.xacro"/>
+      <!-- Instantiate model for the gripper-->
+      <!-- robotiq 2f 85 gripper -->
+      <xacro:robotiq_arg2f_85 prefix=""/>
+    </xacro:if>
+    <!-- If model 140-->
+    <xacro:if value="${gripper_model == 140}">
+      <xacro:include filename="$(find robotiq_2f_140_gripper_visualization)/urdf/robotiq_arg2f_140_model_macro.xacro"/>
+      <!-- Instantiate model for the gripper-->
+      <!-- robotiq 2f 85 gripper -->
+      <xacro:robotiq_arg2f_140 prefix=""/>
+    </xacro:if>
+    <!-- attaches the gripper to the coupler -->
     <joint name="gripper_ur5_joint" type="fixed">
         <parent link="tool0"/>
         <child link="robotiq_arg2f_base_link"/>
-        <origin xyz="0 0 0.01" rpy="0 0 0"/>
+        <origin xyz="0 0 0" rpy="0 0 ${pi/2}"/>
     </joint>
+    <!-- Gazebo grasping plugin -->
+    <!-- Wiki: https://github.com/JenniferBuehler/gazebo-pkgs/wiki/The-Gazebo-grasp-fix-plugin
+    <gazebo>
+      <plugin name="gazebo_grasp_fix" filename="libgazebo_grasp_fix.so">
+            <arm>
+              <arm_name>ur_robot</arm_name>
+              <palm_link> robotiq_arg2f_base_link  </palm_link>
+              <gripper_link> left_inner_finger </gripper_link>
+              <gripper_link> right_inner_finger </gripper_link>
+            </arm>
+          <forces_angle_tolerance>100</forces_angle_tolerance>
+          <update_rate>4</update_rate>
+          <grip_count_threshold>4</grip_count_threshold>
+          <max_grip_count>8</max_grip_count>
+          <release_tolerance>0.005</release_tolerance>
+          <disable_collisions_on_attach>false</disable_collisions_on_attach>
+          <contact_topic>__default_topic__</contact_topic>
+        </plugin>
+    </gazebo>-->
     <!-- Configure self collision properties per link -->
     <gazebo reference="${prefix}shoulder_link">
