Commit message: contact and friction coeffs

File: ur_robot_server/urdf/Robotiq/urRobotiq_macro.xacro (robot description, xacro)
@@ -119,4 +119,45 @@
       </plugin>
     </gazebo>
+    <!-- Better graspping properties-->
+    <gazebo reference="left_inner_finger">
+      <collision>
+        <surface>
+          <contact>
+            <ode>
+            <kp>10000.0</kp>
+            <kd>0.01</kd>
+            <max_vel>0.0</max_vel>
+            <min_depth>0.001</min_depth>
+            </ode>
+          </contact>
+          <friction>
+            <ode>
+            <mu>0.9</mu>
+            <mu2>0.9</mu2>
+            </ode>
+          </friction>
+        </surface>
+      </collision>
+    </gazebo>
+    <gazebo reference="right_inner_finger">
+      <collision>
+        <surface>
+          <contact>
+            <ode>
+            <kp>10000.0</kp>
+            <kd>0.01</kd>
+            <max_vel>0.0</max_vel>
+            <min_depth>0.001</min_depth>
+            </ode>
+          </contact>
+          <friction>
+            <ode>
+            <mu>0.9</mu>
+            <mu2>0.9</mu2>
+            </ode>
+          </friction>
+        </surface>
+      </collision>
+    </gazebo>
     <!-- Configure self collision properties per link -->
     <gazebo reference="${prefix}shoulder_link">

Commit message: removed gripper roll offset

File: ur_robot_server/urdf/Robotiq/urRobotiq_macro.xacro (robot description, xacro)
@@ -93,5 +93,5 @@
         <parent link="tool0"/>
         <child link="robotiq_arg2f_base_link"/>
-        <origin xyz="0 0 0" rpy="0 0 ${pi/2}"/>
+        <origin xyz="0 0 0" rpy="0 0 0"/>
     </joint>
     <!--
